Commit message: 优化修正tf_树

File: cartographer/src/mycarto/urdf/ranger_mini_v2.urdf (robot description, URDF)
Before this commit: robot ranger_mini_v2, 12 links, 11 joints
Links:
- link base_link: geometry collision box size=0.738 0.5 0.338; visual box size=0.738 0.5 0.1
Joints:
- removed joint imu2laser
- added joint imu2robot: type fixed, parent base_link, child imu_link, origin xyz=-0.05 0 0 rpy=0 0 0
- joint base_link_joint: child base_footprint -> base_link; origin xyz=0 0 -0.32 -> xyz=0 0 0.32; parent base_link -> base_footprint
